File: HB-RF-USB/HB-RF-USB.sch (KiCad schematic (older format))
At the start: 22 parts, among them J1 USB_B_Micro, J2 Conn_02x20_Odd_Even, J3 Conn_02x06_Odd_Even, Q1 IRLML6402, Q2 IRLML6402, Q3 IRLML2502, U1 FT232RL

Commit message: - Update to Kicad 5 symbol and footprint libs
- Use different Micro USB Connector for better mechanical stability
Parts:
- C1, C2, C3, C4, C5, C6, C7, C8, C9: footprint Capacitors_SMD:C_0805_HandSoldering -> Capacitor_SMD:C_0805_2012Metric_Pad1.15x1.40mm_HandSolder
- J1: footprint Homebrew:USB-MICRO-MK5P -> Homebrew:U-F-M5DD-Y-1
- J2: footprint Pin_Headers:Pin_Header_Straight_2x20_Pitch2.54mm -> Connector_PinHeader_2.54mm:PinHeader_2x20_P2.54mm_Vertical
- J3: footprint Pin_Headers:Pin_Header_Straight_2x06_Pitch2.54mm -> Connector_PinHeader_2.54mm:PinHeader_2x06_P2.54mm_Vertical
- L1: footprint Inductors_SMD:L_0805_HandSoldering -> Inductor_SMD:L_0805_2012Metric_Pad1.15x1.40mm_HandSolder
- Q1, Q2, Q3: footprint TO_SOT_Packages_SMD:SOT-23_Handsoldering -> Package_TO_SOT_SMD:SOT-23_Handsoldering
- R1, R2, R3, R4, R5: footprint Resistors_SMD:R_0805_HandSoldering -> Resistor_SMD:R_0805_2012Metric_Pad1.15x1.40mm_HandSolder
- U1: footprint Housings_SSOP:SSOP-28_5.3x10.2mm_Pitch0.65mm -> Package_SO:SSOP-28_5.3x10.2mm_P0.65mm; symbol Interface_USB:FT232RL -> HB-RF-USB-rescue:FT232RL-Interface_USB
Changed lines of the file:
@@
 EESchema Schematic File Version 4
 LIBS:HB-RF-USB-cache
-EELAYER 26 0
+EELAYER 30 0
 EELAYER END
 $Descr A4 11693 8268
@@
 $EndDescr
 $Comp
-L Interface_USB:FT232RL U1
+L HB-RF-USB-rescue:FT232RL-Interface_USB U1
 U 1 1 5BDDBC5D
 P 2300 4150
 F 0 "U1" H 2300 5328 50  0000 C CNN
 F 1 "FT232RL" H 2300 5237 50  0000 C CNN
-F 2 "Housings_SSOP:SSOP-28_5.3x10.2mm_Pitch0.65mm" H 2300 4150 50  0001 C CNN
+F 2 "Package_SO:SSOP-28_5.3x10.2mm_P0.65mm" H 2300 4150 50  0001 C CNN
 F 3 "http://www.ftdichip.com/Products/ICs/FT232RL.htm" H 2300 4150 50  0001 C CNN
 	1    2300 4150
@@
 F 0 "J1" H 1105 1767 50  0000 C CNN
 F 1 "USB_B_Micro" H 1105 1676 50  0000 C CNN
-F 2 "Homebrew:USB-MICRO-MK5P" H 1200 1250 50  0001 C CNN
+F 2 "Homebrew:U-F-M5DD-Y-1" H 1200 1250 50  0001 C CNN
 F 3 "~" H 1200 1250 50  0001 C CNN
 	1    1050 1300
@@
 F 0 "J3" H 7550 2017 50  0000 C CNN
 F 1 "Conn_02x06_Odd_Even" H 7550 1926 50  0000 C CNN
-F 2 "Pin_Headers:Pin_Header_Straight_2x06_Pitch2.54mm" H 7500 1600 50  0001 C CNN
+F 2 "Connector_PinHeader_2.54mm:PinHeader_2x06_P2.54mm_Vertical" H 7500 1600 50  0001 C CNN
 F 3 "~" H 7500 1600 50  0001 C CNN
 	1    7500 1600
@@
 F 0 "J2" H 6150 5867 50  0000 C CNN
 F 1 "Conn_02x20_Odd_Even" H 6150 5776 50  0000 C CNN
-F 2 "Pin_Headers:Pin_Header_Straight_2x20_Pitch2.54mm" H 6100 4750 50  0001 C CNN
+F 2 "Connector_PinHeader_2.54mm:PinHeader_2x20_P2.54mm_Vertical" H 6100 4750 50  0001 C CNN
 F 3 "~" H 6100 4750 50  0001 C CNN
 	1    6100 4750
@@
 F 0 "C2" H 4592 1546 50  0000 L CNN
 F 1 "100nF" H 4592 1455 50  0000 L CNN
-F 2 "Capacitors_SMD:C_0805_HandSoldering" H 4500 1500 50  0001 C CNN
+F 2 "Capacitor_SMD:C_0805_2012Metric_Pad1.15x1.40mm_HandSolder" H 4500 1500 50  0001 C CNN
 F 3 "~" H 4500 1500 50  0001 C CNN
 	1    4500 1500
@@
 F 0 "Q2" V 8193 3950 50  0000 C CNN
 F 1 "IRLML6402" V 8102 3950 50  0000 C CNN
-F 2 "TO_SOT_Packages_SMD:SOT-23_Handsoldering" H 8050 3875 50  0001 L CIN
+F 2 "Package_TO_SOT_SMD:SOT-23_Handsoldering" H 8050 3875 50  0001 L CIN
 F 3 "https://www.infineon.com/dgdl/irlml6402pbf.pdf?fileId=5546d462533600a401535668d5c2263c" H 7850 3950 50  0001 L CNN
 	1    7850 3950
@@
 F 0 "C7" H 1992 1646 50  0000 L CNN
 F 1 "10nF" H 1992 1555 50  0000 L CNN
-F 2 "Capacitors_SMD:C_0805_HandSoldering" H 1900 1600 50  0001 C CNN
+F 2 "Capacitor_SMD:C_0805_2012Metric_Pad1.15x1.40mm_HandSolder" H 1900 1600 50  0001 C CNN
 F 3 "~" H 1900 1600 50  0001 C CNN
 	1    1900 1600
@@
 F 0 "R1" V 3504 4850 50  0000 C CNN
 F 1 "10K" V 3595 4850 50  0000 C CNN
-F 2 "Resistors_SMD:R_0805_HandSoldering" H 3700 4850 50  0001 C CNN
+F 2 "Resistor_SMD:R_0805_2012Metric_Pad1.15x1.40mm_HandSolder" H 3700 4850 50  0001 C CNN
 F 3 "~" H 3700 4850 50  0001 C CNN
 	1    3700 4850
@@
 F 0 "R3" H 7791 4254 50  0000 R CNN
 F 1 "1K" H 7791 4345 50  0000 R CNN
-F 2 "Resistors_SMD:R_0805_HandSoldering" H 7850 4300 50  0001 C CNN
+F 2 "Resistor_SMD:R_0805_2012Metric_Pad1.15x1.40mm_HandSolder" H 7850 4300 50  0001 C CNN
 F 3 "~" H 7850 4300 50  0001 C CNN
 	1    7850 4300
@@
 F 0 "C6" H 7492 3996 50  0000 L CNN
 F 1 "100nF" H 7492 3905 50  0000 L CNN
-F 2 "Capacitors_SMD:C_0805_HandSoldering" H 7400 3950 50  0001 C CNN
+F 2 "Capacitor_SMD:C_0805_2012Metric_Pad1.15x1.40mm_HandSolder" H 7400 3950 50  0001 C CNN
 F 3 "~" H 7400 3950 50  0001 C CNN
 	1    7400 3950
@@
 F 0 "C5" H 7142 3996 50  0000 L CNN
 F 1 "100nF" H 7142 3905 50  0000 L CNN
-F 2 "Capacitors_SMD:C_0805_HandSoldering" H 7050 3950 50  0001 C CNN
+F 2 "Capacitor_SMD:C_0805_2012Metric_Pad1.15x1.40mm_HandSolder" H 7050 3950 50  0001 C CNN
 F 3 "~" H 7050 3950 50  0001 C CNN
 	1    7050 3950
@@
 F 0 "Q1" V 6493 1500 50  0000 C CNN
 F 1 "IRLML6402" V 6402 1500 50  0000 C CNN
-F 2 "TO_SOT_Packages_SMD:SOT-23_Handsoldering" H 6350 1425 50  0001 L CIN
+F 2 "Package_TO_SOT_SMD:SOT-23_Handsoldering" H 6350 1425 50  0001 L CIN
 F 3 "https://www.infineon.com/dgdl/irlml6402pbf.pdf?fileId=5546d462533600a401535668d5c2263c" H 6150 1500 50  0001 L CNN
 	1    6150 1500
@@
 F 0 "R2" H 6091 1804 50  0000 R CNN
 F 1 "1K" H 6091 1895 50  0000 R CNN
-F 2 "Resistors_SMD:R_0805_HandSoldering" H 6150 1850 50  0001 C CNN
+F 2 "Resistor_SMD:R_0805_2012Metric_Pad1.15x1.40mm_HandSolder" H 6150 1850 50  0001 C CNN
 F 3 "~" H 6150 1850 50  0001 C CNN
 	1    6150 1850
@@
 F 0 "C3" H 6692 1546 50  0000 L CNN
 F 1 "100nF" H 6692 1455 50  0000 L CNN
-F 2 "Capacitors_SMD:C_0805_HandSoldering" H 6600 1500 50  0001 C CNN
+F 2 "Capacitor_SMD:C_0805_2012Metric_Pad1.15x1.40mm_HandSolder" H 6600 1500 50  0001 C CNN
 F 3 "~" H 6600 1500 50  0001 C CNN
 	1    6600 1500
@@
 F 0 "C4" H 7042 1546 50  0000 L CNN
 F 1 "100nF" H 7042 1455 50  0000 L CNN
-F 2 "Capacitors_SMD:C_0805_HandSoldering" H 6950 1500 50  0001 C CNN
+F 2 "Capacitor_SMD:C_0805_2012Metric_Pad1.15x1.40mm_HandSolder" H 6950 1500 50  0001 C CNN
 F 3 "~" H 6950 1500 50  0001 C CNN
 	1    6950 1500
@@
 F 0 "C1" H 3642 1546 50  0000 L CNN
 F 1 "100nF" H 3642 1455 50  0000 L CNN
-F 2 "Capacitors_SMD:C_0805_HandSoldering" H 3550 1500 50  0001 C CNN
+F 2 "Capacitor_SMD:C_0805_2012Metric_Pad1.15x1.40mm_HandSolder" H 3550 1500 50  0001 C CNN
 F 3 "~" H 3550 1500 50  0001 C CNN
 	1    3550 1500
@@
 F 0 "C8" H 4042 1546 50  0000 L CNN
 F 1 "4.7uF" H 4042 1455 50  0000 L CNN
-F 2 "Capacitors_SMD:C_0805_HandSoldering" H 3950 1500 50  0001 C CNN
+F 2 "Capacitor_SMD:C_0805_2012Metric_Pad1.15x1.40mm_HandSolder" H 3950 1500 50  0001 C CNN
 F 3 "~" H 3950 1500 50  0001 C CNN
 	1    3950 1500
@@
 F 0 "L1" V 1972 1100 50  0000 C CNN
 F 1 "Ferrite Bead" V 2063 1100 50  0000 C CNN
-F 2 "Inductors_SMD:L_0805_HandSoldering" H 2150 1100 50  0001 C CNN
+F 2 "Inductor_SMD:L_0805_2012Metric_Pad1.15x1.40mm_HandSolder" H 2150 1100 50  0001 C CNN
 F 3 "~" H 2150 1100 50  0001 C CNN
 	1    2150 1100
@@
 F 0 "C9" H 1042 2096 50  0000 L CNN
 F 1 "4.7nF" H 1042 2005 50  0000 L CNN
-F 2 "Capacitors_SMD:C_0805_HandSoldering" H 950 2050 50  0001 C CNN
+F 2 "Capacitor_SMD:C_0805_2012Metric_Pad1.15x1.40mm_HandSolder" H 950 2050 50  0001 C CNN
 F 3 "~" H 950 2050 50  0001 C CNN
 	1    950  2050
@@
 F 0 "R4" H 1391 2004 50  0000 R CNN
 F 1 "1M" H 1391 2095 50  0000 R CNN
-F 2 "Resistors_SMD:R_0805_HandSoldering" H 1450 2050 50  0001 C CNN
+F 2 "Resistor_SMD:R_0805_2012Metric_Pad1.15x1.40mm_HandSolder" H 1450 2050 50  0001 C CNN
 F 3 "~" H 1450 2050 50  0001 C CNN
 	1    1450 2050
@@
 F 0 "Q3" V 6350 2900 50  0000 C CNN
 F 1 "IRLML2502" V 6441 2900 50  0000 C CNN
-F 2 "TO_SOT_Packages_SMD:SOT-23_Handsoldering" H 6300 3000 50  0001 C CNN
+F 2 "Package_TO_SOT_SMD:SOT-23_Handsoldering" H 6300 3000 50  0001 C CNN
 F 3 "~" H 6100 2900 50  0001 C CNN
 	1    6100 2900
@@
 F 0 "R5" V 6354 2800 50  0000 C CNN
 F 1 "10K" V 6445 2800 50  0000 C CNN
-F 2 "Resistors_SMD:R_0805_HandSoldering" H 6550 2800 50  0001 C CNN
+F 2 "Resistor_SMD:R_0805_2012Metric_Pad1.15x1.40mm_HandSolder" H 6550 2800 50  0001 C CNN
 F 3 "~" H 6550 2800 50  0001 C CNN
 	1    6550 2800
